File: Kicad/GC - CAN.sch (KiCad schematic (older format))
At the start: 3 parts, among them U4 SN65HVD232

Commit message: changed all componenents to know version
Parts:
- C4: footprint Capacitors_SMD:C_0603 -> Capacitor_SMD:C_0603_1608Metric
- R16: footprint Resistors_SMD:R_0603 -> Resistor_SMD:R_0603_1608Metric
Changed lines of the file:
@@
 F 0 "R16" V 5100 4100 50  0000 C CNN
 F 1 "120R" V 5200 4100 50  0000 C CNN
-F 2 "Resistors_SMD:R_0603" V 5130 4100 30  0001 C CNN
+F 2 "Resistor_SMD:R_0603_1608Metric" V 5130 4100 30  0001 C CNN
 F 3 "" H 5200 4100 30  0000 C CNN
 	1    5200 4100
@@
 F 0 "C4" H 7200 4200 50  0000 L CNN
 F 1 "100nF" H 7206 4015 50  0000 L CNN
-F 2 "Capacitors_SMD:C_0603" H 7238 3950 30  0001 C CNN
+F 2 "Capacitor_SMD:C_0603_1608Metric" H 7238 3950 30  0001 C CNN
 F 3 "" H 7200 4100 60  0000 C CNN
 F 4 "50V" H 7200 4100 50  0001 C CNN "Tension"
