File: Kicad/GC - Driver.sch (KiCad schematic (older format))
At the start: 45 parts, among them U3 DRV8302

Commit message: changed all componenents to know version
Parts:
- C21, C22, C23, C24, C25, C26, C27, C28, C32, C33, C34, C35, C36, C37, C39, C56: footprint Capacitors_SMD:C_0603 -> Capacitor_SMD:C_0603_1608Metric
- C29, C31, C55: footprint Capacitors_SMD:C_1210 -> Capacitor_SMD:C_1210_3225Metric
- C30, C38: footprint Capacitors_SMD:C_0805 -> Capacitor_SMD:C_0805_2012Metric
- C40, C41, C43, C44: footprint Capacitors_SMD:C_1206 -> Capacitor_SMD:C_1206_3216Metric
- R26, R27, R28, R29, R30, R31, R32, R33, R34, R35, R36, R39, R40, R41, R42, R43: footprint Resistors_SMD:R_0603 -> Resistor_SMD:R_0603_1608Metric
