File: Kicad/GC - Hall_Filters.sch (KiCad schematic (older format))
At the start: 11 parts

Commit message: changed all componenents to know version
Parts:
- C5, C6, C7, C8: footprint Capacitors_SMD:C_0603 -> Capacitor_SMD:C_0603_1608Metric
- R18, R19, R20, R21, R23, R24, R25: footprint Resistors_SMD:R_0603 -> Resistor_SMD:R_0603_1608Metric
Changed lines of the file:
@@
 F 0 "R18" V 4850 3450 50  0000 C CNN
 F 1 "10k" V 4900 3250 50  0000 C CNN
-F 2 "Resistors_SMD:R_0603" H 4900 3250 60  0001 C CNN
+F 2 "Resistor_SMD:R_0603_1608Metric" H 4900 3250 60  0001 C CNN
 F 3 "" H 4900 3250 60  0001 C CNN
 	1    4900 3250
@@
 F 0 "R25" V 5500 3950 50  0000 C CNN
 F 1 "10k" V 5550 3750 50  0000 C CNN
-F 2 "Resistors_SMD:R_0603" H 5550 3750 60  0001 C CNN
+F 2 "Resistor_SMD:R_0603_1608Metric" H 5550 3750 60  0001 C CNN
 F 3 "" H 5550 3750 60  0001 C CNN
 	1    5550 3750
@@
 F 0 "R24" V 5500 3850 50  0000 C CNN
 F 1 "10k" V 5550 3650 50  0000 C CNN
-F 2 "Resistors_SMD:R_0603" H 5550 3650 60  0001 C CNN
+F 2 "Resistor_SMD:R_0603_1608Metric" H 5550 3650 60  0001 C CNN
 F 3 "" H 5550 3650 60  0001 C CNN
 	1    5550 3650
@@
 F 0 "R23" V 5500 3750 50  0000 C CNN
 F 1 "10k" V 5550 3550 50  0000 C CNN
-F 2 "Resistors_SMD:R_0603" H 5550 3550 60  0001 C CNN
+F 2 "Resistor_SMD:R_0603_1608Metric" H 5550 3550 60  0001 C CNN
 F 3 "" H 5550 3550 60  0001 C CNN
 	1    5550 3550
@@
 F 0 "R19" V 4950 3450 50  0000 C CNN
 F 1 "2k2" V 5000 3250 50  0000 C CNN
-F 2 "Resistors_SMD:R_0603" H 5000 3250 60  0001 C CNN
+F 2 "Resistor_SMD:R_0603_1608Metric" H 5000 3250 60  0001 C CNN
 F 3 "" H 5000 3250 60  0001 C CNN
 	1    5000 3250
@@
 F 0 "R20" V 5050 3450 50  0000 C CNN
 F 1 "2k2" V 5100 3250 50  0000 C CNN
-F 2 "Resistors_SMD:R_0603" H 5100 3250 60  0001 C CNN
+F 2 "Resistor_SMD:R_0603_1608Metric" H 5100 3250 60  0001 C CNN
 F 3 "" H 5100 3250 60  0001 C CNN
 	1    5100 3250
@@
 F 0 "R21" V 5150 3450 50  0000 C CNN
 F 1 "2k2" V 5200 3250 50  0000 C CNN
-F 2 "Resistors_SMD:R_0603" H 5200 3250 60  0001 C CNN
+F 2 "Resistor_SMD:R_0603_1608Metric" H 5200 3250 60  0001 C CNN
 F 3 "" H 5200 3250 60  0001 C CNN
 	1    5200 3250
@@
 F 0 "C5" H 5600 4300 50  0000 L CNN
 F 1 "4.7nF" H 5600 4100 50  0000 L CNN
-F 2 "Capacitors_SMD:C_0603" H 5550 4200 60  0001 C CNN
+F 2 "Capacitor_SMD:C_0603_1608Metric" H 5550 4200 60  0001 C CNN
 F 3 "" H 5550 4200 60  0001 C CNN
 F 4 "6.3V" H 5550 4200 50  0001 C CNN "Tension"
@@
 F 0 "C8" H 6350 4300 50  0000 L CNN
 F 1 "4.7nF" H 6350 4100 50  0000 L CNN
-F 2 "Capacitors_SMD:C_0603" H 6300 4200 60  0001 C CNN
+F 2 "Capacitor_SMD:C_0603_1608Metric" H 6300 4200 60  0001 C CNN
 F 3 "" H 6300 4200 60  0001 C CNN
 F 4 "6.3V" H 6300 4200 50  0001 C CNN "Tension"
@@
 F 0 "C7" H 6100 4300 50  0000 L CNN
 F 1 "4.7nF" H 6100 4100 50  0000 L CNN
-F 2 "Capacitors_SMD:C_0603" H 6050 4200 60  0001 C CNN
+F 2 "Capacitor_SMD:C_0603_1608Metric" H 6050 4200 60  0001 C CNN
 F 3 "" H 6050 4200 60  0001 C CNN
 F 4 "6.3V" H 6050 4200 50  0001 C CNN "Tension"
@@
 F 0 "C6" H 5850 4300 50  0000 L CNN
 F 1 "4.7nF" H 5850 4100 50  0000 L CNN
-F 2 "Capacitors_SMD:C_0603" H 5800 4200 60  0001 C CNN
+F 2 "Capacitor_SMD:C_0603_1608Metric" H 5800 4200 60  0001 C CNN
 F 3 "" H 5800 4200 60  0001 C CNN
 F 4 "6.3V" H 5800 4200 50  0001 C CNN "Tension"
