File: Kicad/GC - Mosfets.sch (KiCad schematic (older format))
At the start: 15 parts, among them Q1 IRFB7530, Q2 IRFB7530, Q3 IRFB7530, Q4 IRFB7530, Q5 IRFB7530, Q6 IRFB7530

Commit message: changed all componenents to know version
Parts:
- R1, R10, R11, R12, R13, R2, R7, R8, R9: footprint Resistors_SMD:R_0603 -> Resistor_SMD:R_0603_1608Metric
Changed lines of the file:
@@
 F 0 "R13" V 7350 4150 50  0000 C CNN
 F 1 "39k" V 7250 4150 50  0000 C CNN
-F 2 "Resistors_SMD:R_0603" H 7250 4150 60  0001 C CNN
+F 2 "Resistor_SMD:R_0603_1608Metric" H 7250 4150 60  0001 C CNN
 F 3 "" H 7250 4150 60  0001 C CNN
 	1    7250 4150
@@
 F 0 "R7" V 4200 4150 50  0000 C CNN
 F 1 "39k" V 4100 4150 50  0000 C CNN
-F 2 "Resistors_SMD:R_0603" H 4100 4150 60  0001 C CNN
+F 2 "Resistor_SMD:R_0603_1608Metric" H 4100 4150 60  0001 C CNN
 F 3 "" H 4100 4150 60  0001 C CNN
 	1    4100 4150
@@
 F 0 "R2" V 3750 3850 50  0000 C CNN
 F 1 "4R7" V 3650 3850 50  0000 C CNN
-F 2 "Resistors_SMD:R_0603" H 3650 3850 60  0001 C CNN
+F 2 "Resistor_SMD:R_0603_1608Metric" H 3650 3850 60  0001 C CNN
 F 3 "" H 3650 3850 60  0001 C CNN
 	1    3650 3850
@@
 F 0 "R1" V 3750 2900 50  0000 C CNN
 F 1 "4R7" V 3650 2900 50  0000 C CNN
-F 2 "Resistors_SMD:R_0603" H 3650 2900 60  0001 C CNN
+F 2 "Resistor_SMD:R_0603_1608Metric" H 3650 2900 60  0001 C CNN
 F 3 "" H 3650 2900 60  0001 C CNN
 	1    3650 2900
@@
 F 0 "R8" V 5300 2900 50  0000 C CNN
 F 1 "4R7" V 5200 2900 50  0000 C CNN
-F 2 "Resistors_SMD:R_0603" H 5200 2900 60  0001 C CNN
+F 2 "Resistor_SMD:R_0603_1608Metric" H 5200 2900 60  0001 C CNN
 F 3 "" H 5200 2900 60  0001 C CNN
 	1    5200 2900
@@
 F 0 "R9" V 5300 3850 50  0000 C CNN
 F 1 "4R7" V 5200 3850 50  0000 C CNN
-F 2 "Resistors_SMD:R_0603" H 5200 3850 60  0001 C CNN
+F 2 "Resistor_SMD:R_0603_1608Metric" H 5200 3850 60  0001 C CNN
 F 3 "" H 5200 3850 60  0001 C CNN
 	1    5200 3850
@@
 F 0 "R12" V 6900 3850 50  0000 C CNN
 F 1 "4R7" V 6800 3850 50  0000 C CNN
-F 2 "Resistors_SMD:R_0603" H 6800 3850 60  0001 C CNN
+F 2 "Resistor_SMD:R_0603_1608Metric" H 6800 3850 60  0001 C CNN
 F 3 "" H 6800 3850 60  0001 C CNN
 	1    6800 3850
@@
 F 0 "R11" V 6900 2900 50  0000 C CNN
 F 1 "4R7" V 6800 2900 50  0000 C CNN
-F 2 "Resistors_SMD:R_0603" H 6800 2900 60  0001 C CNN
+F 2 "Resistor_SMD:R_0603_1608Metric" H 6800 2900 60  0001 C CNN
 F 3 "" H 6800 2900 60  0001 C CNN
 	1    6800 2900
@@
 F 0 "R10" V 5100 4150 50  0000 C CNN
 F 1 "39k" V 5200 4150 50  0000 C CNN
-F 2 "Resistors_SMD:R_0603" H 5200 4150 60  0001 C CNN
+F 2 "Resistor_SMD:R_0603_1608Metric" H 5200 4150 60  0001 C CNN
 F 3 "" H 5200 4150 60  0001 C CNN
 	1    5200 4150
