File: Kicad/GC - Power.sch (KiCad schematic (older format))
At the start: 18 parts, among them U2 XC6220B331MR, U5 TPS54360DDA

Commit message: changed all componenents to know version
Parts:
- C3, C49, C50: footprint Capacitors_SMD:C_1206 -> Capacitor_SMD:C_1210_3225Metric
- C46, C47, C51, C52, C53: footprint Capacitors_SMD:C_0603 -> Capacitor_SMD:C_0603_1608Metric
- R17, R44, R45, R5: footprint Resistors_SMD:R_0603 -> Resistor_SMD:R_0603_1608Metric
Changed lines of the file:
@@
 F 0 "C46" H 7015 3996 50  0000 L CNN
 F 1 "10uF" H 7015 3905 50  0000 L CNN
-F 2 "Capacitors_SMD:C_0603" H 6900 3950 60  0001 C CNN
+F 2 "Capacitor_SMD:C_0603_1608Metric" H 6900 3950 60  0001 C CNN
 F 3 "" H 6900 3950 60  0001 C CNN
 F 4 "25V" H 6900 3950 50  0001 C CNN "Tension"
@@
 F 0 "C50" H 5000 2250 50  0000 L CNN
 F 1 "10uF" H 4950 2050 50  0000 L CNN
-F 2 "Capacitors_SMD:C_1206" H 5150 2150 60  0001 C CNN
+F 2 "Capacitor_SMD:C_1210_3225Metric" H 5150 2150 60  0001 C CNN
 F 3 "" H 5150 2150 60  0001 C CNN
 F 4 "100V" H 5150 2150 50  0001 C CNN "Tension"
@@
 F 0 "C49" H 4700 2250 50  0000 L CNN
 F 1 "10uF" H 4650 2050 50  0000 L CNN
-F 2 "Capacitors_SMD:C_1206" H 4850 2150 60  0001 C CNN
+F 2 "Capacitor_SMD:C_1210_3225Metric" H 4850 2150 60  0001 C CNN
 F 3 "" H 4850 2150 60  0001 C CNN
 F 4 "100V" H 4850 2150 50  0001 C CNN "Tension"
@@
 F 0 "C3" H 4450 2250 50  0000 L CNN
 F 1 "10uF" H 4350 2050 50  0000 L CNN
-F 2 "Capacitors_SMD:C_1206" H 4550 2150 60  0001 C CNN
+F 2 "Capacitor_SMD:C_1210_3225Metric" H 4550 2150 60  0001 C CNN
 F 3 "" H 4550 2150 60  0001 C CNN
 F 4 "100V" H 4550 2150 50  0001 C CNN "Tension"
@@
 F 0 "C52" H 7250 2350 50  0000 L CNN
 F 1 "51pF" H 7200 2250 50  0000 L CNN
-F 2 "Capacitors_SMD:C_0603" H 7500 2300 60  0001 C CNN
+F 2 "Capacitor_SMD:C_0603_1608Metric" H 7500 2300 60  0001 C CNN
 F 3 "" H 7500 2300 60  0001 C CNN
 F 4 "50V" H 7500 2300 50  0001 C CNN "Tension"
@@
 F 0 "C53" H 7915 2496 50  0000 L CNN
 F 1 "1.8nF" H 7915 2405 50  0000 L CNN
-F 2 "Capacitors_SMD:C_0603" H 7800 2450 60  0001 C CNN
+F 2 "Capacitor_SMD:C_0603_1608Metric" H 7800 2450 60  0001 C CNN
 F 3 "" H 7800 2450 60  0001 C CNN
 F 4 "50V" H 7800 2450 50  0001 C CNN "Tension"
@@
 F 0 "C51" H 6700 1950 50  0000 L CNN
 F 1 "100nF" H 6700 1850 50  0000 L CNN
-F 2 "Capacitors_SMD:C_0603" H 6650 1750 60  0001 C CNN
+F 2 "Capacitor_SMD:C_0603_1608Metric" H 6650 1750 60  0001 C CNN
 F 3 "" H 6650 1750 60  0001 C CNN
 F 4 "50V" H 6650 1750 50  0001 C CNN "Tension"
@@
 F 0 "R45" H 7730 2104 50  0000 R CNN
 F 1 "15.4k" H 7730 2195 50  0000 R CNN
-F 2 "Resistors_SMD:R_0603" V 7730 2150 50  0001 C CNN
+F 2 "Resistor_SMD:R_0603_1608Metric" V 7730 2150 50  0001 C CNN
 F 3 "" H 7800 2150 50  0001 C CNN
 	1    7800 2150
@@
 F 0 "R5" H 5520 2246 50  0000 L CNN
 F 1 "274k" H 5520 2155 50  0000 L CNN
-F 2 "Resistors_SMD:R_0603" V 5380 2200 50  0001 C CNN
+F 2 "Resistor_SMD:R_0603_1608Metric" V 5380 2200 50  0001 C CNN
 F 3 "" H 5450 2200 50  0001 C CNN
 	1    5450 2200
@@
 F 0 "R17" H 7220 2146 50  0000 L CNN
 F 1 "60.4k" H 7220 2055 50  0000 L CNN
-F 2 "Resistors_SMD:R_0603" V 7080 2100 50  0001 C CNN
+F 2 "Resistor_SMD:R_0603_1608Metric" V 7080 2100 50  0001 C CNN
 F 3 "" H 7150 2100 50  0001 C CNN
 	1    7150 2100
@@
 F 0 "R44" H 7220 2496 50  0000 L CNN
 F 1 "11.5k" H 7220 2405 50  0000 L CNN
-F 2 "Resistors_SMD:R_0603" V 7080 2450 50  0001 C CNN
+F 2 "Resistor_SMD:R_0603_1608Metric" V 7080 2450 50  0001 C CNN
 F 3 "" H 7150 2450 50  0001 C CNN
 	1    7150 2450
@@
 F 0 "C47" H 5765 3996 50  0000 L CNN
 F 1 "10uF" H 5765 3905 50  0000 L CNN
-F 2 "Capacitors_SMD:C_0603" H 5650 3950 60  0001 C CNN
+F 2 "Capacitor_SMD:C_0603_1608Metric" H 5650 3950 60  0001 C CNN
 F 3 "" H 5650 3950 60  0001 C CNN
 F 4 "25V" H 5650 3950 50  0001 C CNN "Tension"
