File: Kicad/GC - STM32F4.sch (KiCad schematic (older format))
At the start: 16 parts, among them J9 SWD, U1 STM32F405RGT6, Y2 8MHz

Commit message: gouach logo
Parts:
- J9: symbol conn:Conn_02x03_Odd_Even -> Gouach_Controller-rescue:Conn_02x03_Odd_Even-conn
Changed lines of the file:
@@
 EESchema Schematic File Version 4
+LIBS:Gouach_Controller-cache
 EELAYER 30 0
 EELAYER END
@@
 	7500 5950 7500 6200
 $Comp
-L conn:Conn_02x03_Odd_Even J9
+L Gouach_Controller-rescue:Conn_02x03_Odd_Even-conn J9
 U 1 1 53F77410
 P 9750 3050

Commit message: changed all componenents to know version
Parts:
- C10, C11, C12, C13, C14, C15, C16, C17, C18, C19, C20, C9: footprint Capacitors_SMD:C_0603 -> Capacitor_SMD:C_0603_1608Metric
- R6: footprint Resistors_SMD:R_0603 -> Resistor_SMD:R_0603_1608Metric
Changed lines of the file:
@@
 F 0 "C9" H 7850 1800 50  0000 L CNN
 F 1 "15pF" H 8050 1800 50  0000 L CNN
-F 2 "Capacitors_SMD:C_0603" H 8000 1700 60  0001 C CNN
+F 2 "Capacitor_SMD:C_0603_1608Metric" H 8000 1700 60  0001 C CNN
 F 3 "" H 8000 1700 60  0001 C CNN
 F 4 "50V" H 8000 1700 50  0001 C CNN "Tension"
@@
 F 0 "C15" H 7800 1900 50  0000 L CNN
 F 1 "15pF" H 8050 1900 50  0000 L CNN
-F 2 "Capacitors_SMD:C_0603" H 8000 2000 60  0001 C CNN
+F 2 "Capacitor_SMD:C_0603_1608Metric" H 8000 2000 60  0001 C CNN
 F 3 "" H 8000 2000 60  0001 C CNN
 F 4 "50V" H 8000 2000 50  0001 C CNN "Tension"
@@
 F 0 "C12" H 7550 5650 50  0000 L CNN
 F 1 "100nF" H 7550 5450 50  0000 L CNN
-F 2 "Capacitors_SMD:C_0603" H 7500 5550 60  0001 C CNN
+F 2 "Capacitor_SMD:C_0603_1608Metric" H 7500 5550 60  0001 C CNN
 F 3 "" H 7500 5550 60  0001 C CNN
 F 4 "50V" H 7500 5550 50  0001 C CNN "Tension"
@@
 F 0 "C14" H 7800 5650 50  0000 L CNN
 F 1 "100nF" H 7800 5450 50  0000 L CNN
-F 2 "Capacitors_SMD:C_0603" H 7750 5550 60  0001 C CNN
+F 2 "Capacitor_SMD:C_0603_1608Metric" H 7750 5550 60  0001 C CNN
 F 3 "" H 7750 5550 60  0001 C CNN
 F 4 "50V" H 7750 5550 50  0001 C CNN "Tension"
@@
 F 0 "C13" H 7800 3050 50  0000 L CNN
 F 1 "100nF" H 7800 2850 50  0000 L CNN
-F 2 "Capacitors_SMD:C_0603" H 7750 2950 60  0001 C CNN
+F 2 "Capacitor_SMD:C_0603_1608Metric" H 7750 2950 60  0001 C CNN
 F 3 "" H 7750 2950 60  0001 C CNN
 F 4 "50V" H 7750 2950 50  0001 C CNN "Tension"
@@
 F 0 "C16" H 9450 1400 50  0000 L CNN
 F 1 "100nF" H 9450 1200 50  0000 L CNN
-F 2 "Capacitors_SMD:C_0603" H 9400 1300 60  0001 C CNN
+F 2 "Capacitor_SMD:C_0603_1608Metric" H 9400 1300 60  0001 C CNN
 F 3 "" H 9400 1300 60  0001 C CNN
 F 4 "50V" H 9400 1300 50  0001 C CNN "Tension"
@@
 F 0 "C17" H 9750 1400 50  0000 L CNN
 F 1 "100nF" H 9750 1200 50  0000 L CNN
-F 2 "Capacitors_SMD:C_0603" H 9700 1300 60  0001 C CNN
+F 2 "Capacitor_SMD:C_0603_1608Metric" H 9700 1300 60  0001 C CNN
 F 3 "" H 9700 1300 60  0001 C CNN
 F 4 "50V" H 9700 1300 50  0001 C CNN "Tension"
@@
 F 0 "C20" H 10700 1400 50  0000 L CNN
 F 1 "100nF" H 10700 1200 50  0000 L CNN
-F 2 "Capacitors_SMD:C_0603" H 10650 1300 60  0001 C CNN
+F 2 "Capacitor_SMD:C_0603_1608Metric" H 10650 1300 60  0001 C CNN
 F 3 "" H 10650 1300 60  0001 C CNN
 F 4 "50V" H 10650 1300 50  0001 C CNN "Tension"
@@
 F 0 "C18" H 10050 1400 50  0000 L CNN
 F 1 "100nF" H 10050 1200 50  0000 L CNN
-F 2 "Capacitors_SMD:C_0603" H 10000 1300 60  0001 C CNN
+F 2 "Capacitor_SMD:C_0603_1608Metric" H 10000 1300 60  0001 C CNN
 F 3 "" H 10000 1300 60  0001 C CNN
 F 4 "50V" H 10000 1300 50  0001 C CNN "Tension"
@@
 F 0 "C19" H 10400 1400 50  0000 L CNN
 F 1 "100nF" H 10400 1200 50  0000 L CNN
-F 2 "Capacitors_SMD:C_0603" H 10350 1300 60  0001 C CNN
+F 2 "Capacitor_SMD:C_0603_1608Metric" H 10350 1300 60  0001 C CNN
 F 3 "" H 10350 1300 60  0001 C CNN
 F 4 "50V" H 10350 1300 50  0001 C CNN "Tension"
@@
 F 0 "R6" V 7350 2350 50  0000 C CNN
 F 1 "10k" V 7250 2350 50  0000 C CNN
-F 2 "Resistors_SMD:R_0603" V 7180 2350 50  0001 C CNN
+F 2 "Resistor_SMD:R_0603_1608Metric" V 7180 2350 50  0001 C CNN
 F 3 "" H 7250 2350 50  0001 C CNN
 	1    7250 2350
@@
 F 0 "C11" H 7350 6300 50  0000 L CNN
 F 1 "2.2uF" H 7350 6100 50  0000 L CNN
-F 2 "Capacitors_SMD:C_0603" H 7300 6200 60  0001 C CNN
+F 2 "Capacitor_SMD:C_0603_1608Metric" H 7300 6200 60  0001 C CNN
 F 3 "" H 7300 6200 60  0001 C CNN
 F 4 "25V" H 7300 6200 50  0001 C CNN "Tension"
@@
 F 0 "C10" H 7350 6050 50  0000 L CNN
 F 1 "2.2uF" H 7350 5850 50  0000 L CNN
-F 2 "Capacitors_SMD:C_0603" H 7300 5950 60  0001 C CNN
+F 2 "Capacitor_SMD:C_0603_1608Metric" H 7300 5950 60  0001 C CNN
 F 3 "" H 7300 5950 60  0001 C CNN
 F 4 "25V" H 7300 5950 50  0001 C CNN "Tension"
