File: Kicad/GC - Temp_Sensor.sch (KiCad schematic (older format))
At the start: 3 parts

Commit message: changed all componenents to know version
Parts:
- C1: footprint Capacitors_SMD:C_0603 -> Capacitor_SMD:C_0603_1608Metric
- R14, R15: footprint Resistors_SMD:R_0603 -> Resistor_SMD:R_0603_1608Metric
Changed lines of the file:
@@
 F 0 "R15" V 6000 4200 50  0000 C CNN
 F 1 "10k" V 6100 4200 50  0000 C CNN
-F 2 "Resistors_SMD:R_0603" V 5930 4200 30  0001 C CNN
+F 2 "Resistor_SMD:R_0603_1608Metric" V 5930 4200 30  0001 C CNN
 F 3 "" H 6000 4200 30  0000 C CNN
 	1    6000 4200
@@
 F 0 "C1" H 5750 4300 50  0000 L CNN
 F 1 "2.2uF" H 5756 4115 50  0000 L CNN
-F 2 "Capacitors_SMD:C_0603" H 5788 4050 30  0001 C CNN
+F 2 "Capacitor_SMD:C_0603_1608Metric" H 5788 4050 30  0001 C CNN
 F 3 "" H 5750 4200 60  0000 C CNN
 F 4 "25V" H 5750 4200 50  0001 C CNN "Tension"
@@
 F 0 "R14" V 6000 3800 50  0000 C CNN
 F 1 "NTC 10k" V 6100 3800 50  0000 C CNN
-F 2 "Resistors_SMD:R_0603" V 5930 3800 30  0001 C CNN
+F 2 "Resistor_SMD:R_0603_1608Metric" V 5930 3800 30  0001 C CNN
 F 3 "" H 6000 3800 30  0000 C CNN
 	1    6000 3800
