File: Kicad/Gouach_Controller.sch (KiCad schematic (older format))
At the start: 27 parts, among them J1 HALL/Encoder, J10 USB, J11 CAN, J12 Serial, J2 Peripherals, J3 Peripherals, J4 IN+, J5 IN-, J6 MOTOR3, J7 MOTOR2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

Commit message: gouach logo
Parts:
- J1: symbol conn:Conn_01x06 -> Gouach_Controller-rescue:Conn_01x06-conn
- J10, J12: symbol conn:Conn_01x04 -> Gouach_Controller-rescue:Conn_01x04-conn
- J11: symbol conn:Conn_01x02 -> Gouach_Controller-rescue:Conn_01x02-conn
- J2, J3: symbol conn:Conn_01x07 -> Gouach_Controller-rescue:Conn_01x07-conn
- J4, J5, J6, J7, J8: symbol conn:Conn_01x01 -> Gouach_Controller-rescue:Conn_01x01-conn
Changed lines of the file:
@@
 EESchema Schematic File Version 4
+LIBS:Gouach_Controller-cache
 EELAYER 30 0
 EELAYER END
@@
 $EndSheet
 $Comp
-L conn:Conn_01x01 J5
+L Gouach_Controller-rescue:Conn_01x01-conn J5
 U 1 1 53FA5B63
 P 9050 1450
@@
 $EndComp
 $Comp
-L conn:Conn_01x01 J4
+L Gouach_Controller-rescue:Conn_01x01-conn J4
 U 1 1 53FA5B6A
 P 9050 1300
@@
 $EndComp
 $Comp
-L conn:Conn_01x01 J6
+L Gouach_Controller-rescue:Conn_01x01-conn J6
 U 1 1 53FA5B71
 P 10250 2850
@@
 $EndComp
 $Comp
-L conn:Conn_01x01 J7
+L Gouach_Controller-rescue:Conn_01x01-conn J7
 U 1 1 53FA5B78
 P 10250 3000
@@
 $EndComp
 $Comp
-L conn:Conn_01x01 J8
+L Gouach_Controller-rescue:Conn_01x01-conn J8
 U 1 1 53FA5B7F
 P 10250 3550
@@
 	8650 1700 8650 1000
 $Comp
-L conn:Conn_01x02 J11
+L Gouach_Controller-rescue:Conn_01x02-conn J11
 U 1 1 540360D1
 P 1350 2850
@@
 $EndComp
 $Comp
-L power:+5V #PWR0107
-U 1 1 5F1616E5
-P 1550 4200
-F 0 "#PWR0107" H 1550 4050 50  0001 C CNN
-F 1 "+5V" H 1550 4350 50  0000 C CNN
-F 2 "" H 1550 4200 50  0001 C CNN
-F 3 "" H 1550 4200 50  0001 C CNN
-	1    1550 4200
-	1    0    0    -1
-$EndComp
-$Comp
 L power:+5V #PWR0109
 U 1 1 5F1602A3
@@
 	7250 1650 7250 1600
 $Comp
-L conn:Conn_01x06 J1
+L Gouach_Controller-rescue:Conn_01x06-conn J1
 U 1 1 522DA047
 P 1350 3550
@@
 	1550 4300 3250 4300
 $Comp
-L conn:Conn_01x04 J12
+L Gouach_Controller-rescue:Conn_01x04-conn J12
 U 1 1 5E47FB07
 P 1350 6000
@@
 $EndComp
 $Comp
-L conn:Conn_01x04 J10
+L Gouach_Controller-rescue:Conn_01x04-conn J10
 U 1 1 5E4E3243
 P 1350 1900
@@
 $EndComp
 $Comp
-L conn:Conn_01x07 J3
+L Gouach_Controller-rescue:Conn_01x07-conn J3
 U 1 1 5E552A33
 P 1350 5200
@@
 	1    1550 5500
 	1    0    0    -1
-$EndComp
-$Comp
-L conn:Conn_01x07 J2
-U 1 1 5E52A003
-P 1350 4500
-F 0 "J2" H 1350 4900 60  0000 C CNN
-F 1 "Peripherals" V 1450 4450 60  0000 C CNN
-F 2 "Romain:TerminalBlock_Phoenix_MPT-2.54mm_7pol" H 1350 4500 60  0001 C CNN
-F 3 "" H 1350 4500 60  0001 C CNN
-	1    1350 4500
-	-1   0    0    -1
 $EndComp
 $Comp
@@
 Wire Wire Line
 	1800 3600 1950 3600
+$Comp
+L power:+5V #PWR0107
+U 1 1 5F1616E5
+P 1550 4200
+F 0 "#PWR0107" H 1550 4050 50  0001 C CNN
+F 1 "+5V" H 1550 4350 50  0000 C CNN
+F 2 "" H 1550 4200 50  0001 C CNN
+F 3 "" H 1550 4200 50  0001 C CNN
+	1    1550 4200
+	1    0    0    -1
+$EndComp
+$Comp
+L Gouach_Controller-rescue:Conn_01x07-conn J2
+U 1 1 5E52A003
+P 1350 4500
+F 0 "J2" H 1350 4900 60  0000 C CNN
+F 1 "Peripherals" V 1450 4450 60  0000 C CNN
+F 2 "Romain:TerminalBlock_Phoenix_MPT-2.54mm_7pol" H 1350 4500 60  0001 C CNN
+F 3 "" H 1350 4500 60  0001 C CNN
+	1    1350 4500
+	-1   0    0    -1
+$EndComp
 $EndSCHEMATC

Commit message: changed all componenents to know version
Parts:
- added U7: picto, logos:picto, symbol gouach_components:picto
- added U8: logo, logos:logotype, symbol gouach_components:logo
- C2: footprint Capacitors_SMD:C_0603 -> Capacitor_SMD:C_0603_1608Metric
- R22, R3, R37, R38, R4, R46, R47: footprint Resistors_SMD:R_0603 -> Resistor_SMD:R_0603_1608Metric
Changed lines of the file:
@@
 F 0 "R4" V 6850 1550 50  0000 C CNN
 F 1 "2k2" V 6900 1750 50  0000 C CNN
-F 2 "Resistors_SMD:R_0603" H 6900 1750 60  0001 C CNN
+F 2 "Resistor_SMD:R_0603_1608Metric" H 6900 1750 60  0001 C CNN
 F 3 "" H 6900 1750 60  0001 C CNN
 	1    6900 1750
@@
 F 0 "R3" V 6850 1450 50  0000 C CNN
 F 1 "39k" V 6900 1650 50  0000 C CNN
-F 2 "Resistors_SMD:R_0603" H 6900 1650 60  0001 C CNN
+F 2 "Resistor_SMD:R_0603_1608Metric" H 6900 1650 60  0001 C CNN
 F 3 "" H 6900 1650 60  0001 C CNN
 	1    6900 1650
@@
 F 0 "R38" V 6050 6100 50  0000 C CNN
 F 1 "100R" V 6150 6100 50  0000 C CNN
-F 2 "Resistors_SMD:R_0603" H 6150 6100 60  0001 C CNN
+F 2 "Resistor_SMD:R_0603_1608Metric" H 6150 6100 60  0001 C CNN
 F 3 "" H 6150 6100 60  0001 C CNN
 	1    6150 6100
@@
 F 0 "R37" V 6050 5800 50  0000 C CNN
 F 1 "100R" V 6150 5800 50  0000 C CNN
-F 2 "Resistors_SMD:R_0603" H 6150 5800 60  0001 C CNN
+F 2 "Resistor_SMD:R_0603_1608Metric" H 6150 5800 60  0001 C CNN
 F 3 "" H 6150 5800 60  0001 C CNN
 	1    6150 5800
@@
 F 0 "R22" V 6050 5500 50  0000 C CNN
 F 1 "2k2" V 6150 5500 50  0000 C CNN
-F 2 "Resistors_SMD:R_0603" H 6150 5500 60  0001 C CNN
+F 2 "Resistor_SMD:R_0603_1608Metric" H 6150 5500 60  0001 C CNN
 F 3 "" H 6150 5500 60  0001 C CNN
 	1    6150 5500
@@
 F 0 "C2" V 6850 1950 50  0000 L CNN
 F 1 "100nF" V 6850 1600 50  0000 L CNN
-F 2 "Capacitors_SMD:C_0603" H 6900 1900 60  0001 C CNN
+F 2 "Capacitor_SMD:C_0603_1608Metric" H 6900 1900 60  0001 C CNN
 F 3 "" H 6900 1900 60  0001 C CNN
 F 4 "50V" H 6900 1900 50  0001 C CNN "Tension"
@@
 F 0 "R46" V 2850 5550 50  0000 C CNN
 F 1 "100R" V 2950 5550 50  0000 C CNN
-F 2 "Resistors_SMD:R_0603" H 2950 5550 60  0001 C CNN
+F 2 "Resistor_SMD:R_0603_1608Metric" H 2950 5550 60  0001 C CNN
 F 3 "" H 2950 5550 60  0001 C CNN
 	1    2950 5550
@@
 F 0 "R47" V 2850 5750 50  0000 C CNN
 F 1 "10k" V 2950 5750 50  0000 C CNN
-F 2 "Resistors_SMD:R_0603" H 2950 5750 60  0001 C CNN
+F 2 "Resistor_SMD:R_0603_1608Metric" H 2950 5750 60  0001 C CNN
 F 3 "" H 2950 5750 60  0001 C CNN
 	1    2950 5750
@@
 	-1   0    0    -1
 $EndComp
+$Comp
+L Graphic:Logo_Open_Hardware_Small #LOGO1
+U 1 1 5E70AD78
+P 9450 5300
+F 0 "#LOGO1" H 9450 5575 50  0001 C CNN
+F 1 "Logo_Open_Hardware_Small" H 9450 5075 50  0001 C CNN
+F 2 "logos:picto" H 9450 5300 50  0001 C CNN
+F 3 "~" H 9450 5300 50  0001 C CNN
+	1    9450 5300
+	1    0    0    -1
+$EndComp
+$Comp
+L gouach_components:picto U7
+U 1 1 5E728F61
+P 9400 5750
+F 0 "U7" H 9425 5796 50  0000 L CNN
+F 1 "picto" H 9425 5705 50  0000 L CNN
+F 2 "logos:picto" H 9400 5750 50  0001 C CNN
+F 3 "" H 9400 5750 50  0001 C CNN
+	1    9400 5750
+	1    0    0    -1
+$EndComp
+$Comp
+L gouach_components:logo U8
+U 1 1 5E7299A7
+P 9450 6000
+F 0 "U8" H 9475 6046 50  0000 L CNN
+F 1 "logo" H 9475 5955 50  0000 L CNN
+F 2 "logos:logotype" H 9450 6000 50  0001 C CNN
+F 3 "" H 9450 6000 50  0001 C CNN
+	1    9450 6000
+	1    0    0    -1
+$EndComp
 $EndSCHEMATC

Commit message: Modified silkscreens. Changed peripheral connectors. Fixed some 3D libs paths
Parts:
- J2, J3: footprint Romain:TerminalBlock_Phoenix_MPT-2.54mm_7pol -> Connector_PinHeader_2.54mm:PinHeader_1x06_P2.54mm_Vertical; symbol Gouach_Controller-rescue:Conn_01x07-conn -> Gouach_Controller-rescue:Conn_01x06-conn
- U7: symbol gouach_components:picto -> Gouach_Controller-rescue:picto-gouach_components
- U8: symbol gouach_components:logo -> Gouach_Controller-rescue:logo-gouach_components
Connections:
- net +5V: now also J2.3 (Pin_3), J3.1 (Pin_1); no longer J2.1 (Pin_1), J2.4 (Pin_4), J3.2 (Pin_2)
- net ADC_BRAKE: now also J3.3 (Pin_3); no longer J3.4 (Pin_4)
- net ADC_THROTTLE: now also J2.1 (Pin_1); no longer J2.2 (Pin_2)
- net ADC_TORQUE: now also J2.5 (Pin_5); no longer J2.6 (Pin_6)
- net CRUISE: now also J2.6 (Pin_6); no longer J2.7 (Pin_7)
- net GND: now also J2.2 (Pin_2), J3.4 (Pin_4), J3.6 (Pin_6); no longer J2.3 (Pin_3), J3.1 (Pin_1), J3.5 (Pin_5), J3.7 (Pin_7)
- net IO_BRAKE: now also J3.2 (Pin_2); no longer J3.3 (Pin_3)
- net PFS: now also J2.4 (Pin_4); no longer J2.5 (Pin_5)
- net at Q7.2 (S): now also J3.5 (Pin_5); no longer J3.6 (Pin_6)
Changed lines of the file:
@@
 EESchema Schematic File Version 4
-LIBS:Gouach_Controller-cache
 EELAYER 30 0
 EELAYER END
@@
 $EndComp
 $Comp
-L power:GND #PWR0123
-U 1 1 5F199967
-P 1550 4400
-F 0 "#PWR0123" H 1550 4150 50  0001 C CNN
-F 1 "GND" V 1550 4200 50  0000 C CNN
-F 2 "" H 1550 4400 50  0001 C CNN
-F 3 "" H 1550 4400 50  0001 C CNN
-	1    1550 4400
-	0    -1   -1   0
-$EndComp
-$Comp
 L power:GND #PWR0124
 U 1 1 5F19975B
@@
 F36 "LAMP_CMD" O L 3250 5550 50
 $EndSheet
-Wire Wire Line
-	1550 4300 3250 4300
 $Comp
 L Gouach_Controller-rescue:Conn_01x04-conn J12
@@
 	6550 1900 5800 1900
 Connection ~ 6550 1900
-$Comp
-L power:+5V #PWR01
-U 1 1 5E4B019E
-P 1550 4500
-F 0 "#PWR01" H 1550 4350 50  0001 C CNN
-F 1 "+5V" V 1550 4700 50  0000 C CNN
-F 2 "" H 1550 4500 50  0001 C CNN
-F 3 "" H 1550 4500 50  0001 C CNN
-	1    1550 4500
-	0    1    1    0
-$EndComp
-$Comp
-L power:GND #PWR02
-U 1 1 5E4B0796
-P 1550 4900
-F 0 "#PWR02" H 1550 4650 50  0001 C CNN
-F 1 "GND" V 1550 4700 50  0000 C CNN
-F 2 "" H 1550 4900 50  0001 C CNN
-F 3 "" H 1550 4900 50  0001 C CNN
-	1    1550 4900
-	0    -1   -1   0
-$EndComp
-Wire Wire Line
-	1550 4700 3250 4700
-Wire Wire Line
-	1550 4600 3250 4600
-Wire Wire Line
-	1550 4800 3250 4800
 Text Label 2200 4600 0    40   ~ 0
 PFS
 Text Label 2200 4800 0    40   ~ 0
 CRUISE
-$Comp
-L power:+5V #PWR05
-U 1 1 5E4E1CA3
-P 1550 5000
-F 0 "#PWR05" H 1550 4850 50  0001 C CNN
-F 1 "+5V" V 1550 5200 50  0000 C CNN
-F 2 "" H 1550 5000 50  0001 C CNN
-F 3 "" H 1550 5000 50  0001 C CNN
-	1    1550 5000
-	0    1    1    0
-$EndComp
-$Comp
-L power:GND #PWR06
-U 1 1 5E4E213F
-P 1550 5300
-F 0 "#PWR06" H 1550 5050 50  0001 C CNN
-F 1 "GND" V 1550 5100 50  0000 C CNN
-F 2 "" H 1550 5300 50  0001 C CNN
-F 3 "" H 1550 5300 50  0001 C CNN
-	1    1550 5300
-	0    -1   -1   0
-$EndComp
-Wire Wire Line
-	1550 5100 3250 5100
-Wire Wire Line
-	1550 5200 3250 5200
 Wire Wire Line
 	6000 5500 5950 5500
@@
 $EndComp
 $Comp
-L Gouach_Controller-rescue:Conn_01x07-conn J3
-U 1 1 5E552A33
-P 1350 5200
-F 0 "J3" H 1350 4800 60  0000 C CNN
-F 1 "Peripherals" V 1450 5150 60  0000 C CNN
-F 2 "Romain:TerminalBlock_Phoenix_MPT-2.54mm_7pol" H 1350 5200 60  0001 C CNN
-F 3 "" H 1350 5200 60  0001 C CNN
-	1    1350 5200
-	-1   0    0    -1
-$EndComp
-$Comp
-L power:GND #PWR0108
-U 1 1 5E554A00
-P 1550 5500
-F 0 "#PWR0108" H 1550 5250 50  0001 C CNN
-F 1 "GND" H 1550 5350 50  0000 C CNN
-F 2 "" H 1550 5500 50  0001 C CNN
-F 3 "" H 1550 5500 50  0001 C CNN
-	1    1550 5500
-	1    0    0    -1
-$EndComp
-$Comp
 L Power_Protection:USBLC6-2SC6 U6
 U 1 1 5E4EB6A7
@@
 	1    0    0    -1
 $EndComp
-Wire Wire Line
-	1550 5400 1750 5400
 Wire Wire Line
 	1750 5400 1750 5850
@@
 	1800 3600 1950 3600
 $Comp
-L power:+5V #PWR0107
-U 1 1 5F1616E5
-P 1550 4200
-F 0 "#PWR0107" H 1550 4050 50  0001 C CNN
-F 1 "+5V" H 1550 4350 50  0000 C CNN
-F 2 "" H 1550 4200 50  0001 C CNN
-F 3 "" H 1550 4200 50  0001 C CNN
-	1    1550 4200
-	1    0    0    -1
-$EndComp
-$Comp
-L Gouach_Controller-rescue:Conn_01x07-conn J2
-U 1 1 5E52A003
-P 1350 4500
-F 0 "J2" H 1350 4900 60  0000 C CNN
-F 1 "Peripherals" V 1450 4450 60  0000 C CNN
-F 2 "Romain:TerminalBlock_Phoenix_MPT-2.54mm_7pol" H 1350 4500 60  0001 C CNN
-F 3 "" H 1350 4500 60  0001 C CNN
-	1    1350 4500
-	-1   0    0    -1
-$EndComp
-$Comp
 L Graphic:Logo_Open_Hardware_Small #LOGO1
 U 1 1 5E70AD78
@@
 $EndComp
 $Comp
-L gouach_components:picto U7
+L Gouach_Controller-rescue:picto-gouach_components U7
 U 1 1 5E728F61
 P 9400 5750
@@
 $EndComp
 $Comp
-L gouach_components:logo U8
+L Gouach_Controller-rescue:logo-gouach_components U8
 U 1 1 5E7299A7
 P 9450 6000
@@
 	1    0    0    -1
 $EndComp
+$Comp
+L Gouach_Controller-rescue:Conn_01x06-conn J2
+U 1 1 5E52A003
+P 1900 4500
+F 0 "J2" H 1900 4900 60  0000 C CNN
+F 1 "Peripherals" V 2000 4450 60  0000 C CNN
+F 2 "Connector_PinHeader_2.54mm:PinHeader_1x06_P2.54mm_Vertical" H 1900 4500 60  0001 C CNN
+F 3 "" H 1900 4500 60  0001 C CNN
+	1    1900 4500
+	-1   0    0    -1
+$EndComp
+Wire Wire Line
+	1300 5400 1750 5400
+$Comp
+L Gouach_Controller-rescue:Conn_01x06-conn J3
+U 1 1 5E552A33
+P 1100 5200
+F 0 "J3" H 1100 4800 60  0000 C CNN
+F 1 "Peripherals" V 1200 5150 60  0000 C CNN
+F 2 "Connector_PinHeader_2.54mm:PinHeader_1x06_P2.54mm_Vertical" H 1100 5200 60  0001 C CNN
+F 3 "" H 1100 5200 60  0001 C CNN
+	1    1100 5200
+	-1   0    0    -1
+$EndComp
+Wire Wire Line
+	1300 5200 3250 5200
+Wire Wire Line
+	1300 5100 3250 5100
+$Comp
+L power:GND #PWR06
+U 1 1 5E4E213F
+P 1300 5300
+F 0 "#PWR06" H 1300 5050 50  0001 C CNN
+F 1 "GND" V 1300 5100 50  0000 C CNN
+F 2 "" H 1300 5300 50  0001 C CNN
+F 3 "" H 1300 5300 50  0001 C CNN
+	1    1300 5300
+	0    -1   -1   0
+$EndComp
+$Comp
+L power:+5V #PWR05
+U 1 1 5E4E1CA3
+P 1300 5000
+F 0 "#PWR05" H 1300 4850 50  0001 C CNN
+F 1 "+5V" V 1300 5200 50  0000 C CNN
+F 2 "" H 1300 5000 50  0001 C CNN
+F 3 "" H 1300 5000 50  0001 C CNN
+	1    1300 5000
+	0    1    1    0
+$EndComp
+Wire Wire Line
+	2100 4800 3250 4800
+Wire Wire Line
+	2100 4600 3250 4600
+Wire Wire Line
+	2100 4700 3250 4700
+$Comp
+L power:+5V #PWR01
+U 1 1 5E4B019E
+P 2100 4500
+F 0 "#PWR01" H 2100 4350 50  0001 C CNN
+F 1 "+5V" V 2100 4700 50  0000 C CNN
+F 2 "" H 2100 4500 50  0001 C CNN
+F 3 "" H 2100 4500 50  0001 C CNN
+	1    2100 4500
+	0    1    1    0
+$EndComp
+Wire Wire Line
+	2100 4300 3250 4300
+$Comp
+L power:GND #PWR0123
+U 1 1 5F199967
+P 2100 4400
+F 0 "#PWR0123" H 2100 4150 50  0001 C CNN
+F 1 "GND" V 2100 4200 50  0000 C CNN
+F 2 "" H 2100 4400 50  0001 C CNN
+F 3 "" H 2100 4400 50  0001 C CNN
+	1    2100 4400
+	0    -1   -1   0
+$EndComp
+$Comp
+L power:GND #PWR0108
+U 1 1 5E554A00
+P 1300 5500
+F 0 "#PWR0108" H 1300 5250 50  0001 C CNN
+F 1 "GND" H 1300 5350 50  0000 C CNN
+F 2 "" H 1300 5500 50  0001 C CNN
+F 3 "" H 1300 5500 50  0001 C CNN
+	1    1300 5500
+	0    -1   -1   0
+$EndComp
 $EndSCHEMATC
